File: kicad_source/RS485-Power-Injector/RS485-Power-Injector.kicad_pcb (KiCad board)
At the start: 2 copper layers, 38 x 55 mm, 28 parts, among them J1 PowerPole, J2 DNI, J3 DNI, J4 SM04B-GHS-TB, J5 EH_S4B-EH, J6 EH_S4B-EH, J7 DNI, U1 L78L05_SOT89, U2 SN75176AD

Commit message: Rename from l3xz-hw-rs485-power-injector to RS485-Power-Injector. (#7)
Other:
- board text added: "RS485-Power-Injector 0.1"
- board text added: "https://github.com/107-systems/ RS485-Power-Injector"
- board text removed: "https://github.com/107-systems/ l3xz-hw-rs485-power-injector"
- board text removed: "l3xz-hw-rs485-power-injector 0.1"
