File: kicad_source/RS485-Power-Injector/RS485-Power-Injector.kicad_sch (KiCad schematic)
At the start: 28 parts, among them J1 PowerPole, J2 DNI, J3 DNI, J4 SM04B-GHS-TB, J5 EH_S4B-EH, J6 EH_S4B-EH, J7 DNI, U1 L78L05_SOT89, U2 SN75176AD

Commit message: Rename from l3xz-hw-rs485-power-injector to RS485-Power-Injector. (#7)
Other:
- title: l3xz-hw-rs485-power-injector -> RS485-Power-Injector
Changed lines of the file:
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@@
   (paper "A4")
   (title_block
-    (title "l3xz-hw-rs485-power-injector")
+    (title "RS485-Power-Injector")
     (date "2023-01-23")
     (rev "0.1")
